File: hardware/Central_Unit/central-unit-hub.kicad_sch (KiCad schematic)
At the start: 4 parts

Commit message: v1.9: Minor Fixes
Parts:
- BT1: renamed from BT; value 3.7V Li-Po 1000mAh -> AKY0571 + MOLEX 51021-0200
- U1: renamed from U; value Beetle ESP32-C6 -> DFR1117
- renumbered BZ to BZ1, D to D1
Other:
- note removed: "Components: DFRobot Beetle ESP32-C6 / 3.7V 1000mAh Li-Po Battery / LED Diffused 5mm RGB Programmable WS2812D / Buzzer 2-5V 30mA"
- note removed: "v2: Components updated. Wiring added. Revisions may occur."
- moved on the sheet: BT1, BZ1, D1
