File: hardware/Peripheral_Unit/peripheral-unit.kicad_sch (KiCad schematic)
At the start: 8 parts, among them J1 Conn_01x08, J2 Conn_01x03, J3 Conn_01x02, U1 ESP32-H2-MINI-1-H2, U2 TPS22860DBVR, U3 LP2985-3.3

Commit message: v1.7: Minor Fixes
Parts:
- removed U3: LP2985-3.3, Package_TO_SOT_SMD:SOT-23-5, symbol Regulator_Linear:LP2985-3.3
- added U3: TPS7A0212PDBVR, SOT23_DBV_TEX, symbol TPS7A0212PDVR:TPS7A0212PDBVR
- BT: value Li-SOCl2 19000 mAh Battery -> ER34615
- C: value Capacitor -> 6TPB470M
- J1: value Conn_01x08 -> XM125
- J2: value Conn_01x03 -> EKMB1101111
- J3: value Conn_01x02 -> S12B-PH-K-S(LF)(SN)
- U1: value ESP32-H2-MINI-1-H2 -> ESP32-H2-Zero; footprint ESP32-H2-MINI-1-H2:MODULE_ESP32-H2-MINI-1-H2 -> (none)
Connections:
- net GND: now also U3.2 (GND)
- net at BT.1 (+), C.1: now also U3.1 (IN)
Other:
- note added: "30-07-26"
- note removed: "09-07-26"
- note removed: "3.3V LDO Regulator"
- note removed: "Components: Waveshare ESP32-H2-Zero / EVE Energy ER34615 D-size Li-SOCl2 19000mAh Battery / low-ESR Tantalum capacitor or Solid Polymer capacitor (470-1000μF & 6.3V or 10V)"
- note removed: "JST-PH Power Input"
- note removed: "PIR Sensor Interface"
- note removed: "Power Gating Load Switch"
- note removed: "mmWave Radar Interface"
- note removed: "v2: Components updated. Wiring added."
- moved on the sheet: J3, U2

Commit message: v1.8: Minor Fixes
Parts:
- removed U1: ESP32-H2-Zero, symbol ESP32-H2-MINI-1-H2:ESP32-H2-MINI-1-H2
- added U1: MDBT50Q-P1M, RF_Module:Raytac_MDBT50Q, symbol RF_Module:MDBT50Q-P1MV2
- U3: value TPS7A0212PDBVR -> TPS7A0233PDBVR
Connections:
- net GND: no longer BT.2 (-), C.2
- new net: U1.1 (GND), U1.15 (GND), U1.2 (GND), U1.33 (GND), U1.55 (GND)
- now unconnected: BT.1 (+), C.1, U3.1 (IN)

Commit message: v1.9: Minor Fixes
Other:
- moved on the sheet: J3
Changed lines of the file:
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@@
 	(symbol
 		(lib_id "Connector_Generic:Conn_01x02")
-		(at 100.33 124.46 0)
+		(at 100.33 132.08 0)
 		(unit 1)
 		(body_style 1)
@@
 		(fields_autoplaced yes)
 		(property "Reference" "J3"
-			(at 102.87 123.1899 0)
+			(at 102.87 130.8099 0)
 			(show_name no)
 			(do_not_autoplace no)
@@
 		)
 		(property "Value" "S12B-PH-K-S(LF)(SN)"
-			(at 102.87 125.7299 0)
+			(at 102.87 133.3499 0)
 			(show_name no)
 			(do_not_autoplace no)
@@
 		)
 		(property "Footprint" ""
-			(at 100.33 124.46 0)
+			(at 100.33 132.08 0)
 			(hide yes)
 			(show_name no)
@@
 		)
 		(property "Datasheet" ""
-			(at 100.33 124.46 0)
+			(at 100.33 132.08 0)
 			(hide yes)
 			(show_name no)
@@
 		)
 		(property "Description" "JST-PH Power Input"
-			(at 102.87 128.2699 0)
+			(at 102.87 135.8899 0)
 			(show_name no)
 			(do_not_autoplace no)

Commit message: Add files via upload
Parts:
- removed J3: S12B-PH-K-S(LF)(SN), symbol Connector_Generic:Conn_01x02
- added J3: Conn_01x09, symbol Connector_Generic:Conn_01x09
- added J4: Conn_01x06, Connector_JST:JST_PH_B6B-PH-K_1x06_P2.00mm_Vertical, symbol Connector_Generic:Conn_01x06
- added R1, R2: 100kΩ, symbol Device:R
- added SW1: SW_SPST, symbol Switch:SW_SPST
- added U4: TPS7A0218PDBVR, SOT23_DBV_TEX, symbol TPS7A0212PDVR:TPS7A0212PDBVR
Connections:
- net GND: now also BT.2 (-), C.2, J1.10 (GND), J1.13 (GND), J1.16 (GND), J1.19 (GND), J1.2 (GND), J1.22 (GND), J1.27 (GND), J1.4 (GND), J1.7 (GND), J2.3 (Pin_3), U1.1 (GND), U1.15 (GND), U1.2 (GND), U1.33 (GND), U1.55 (GND), U2.2 (GND), J3.1 (GND), J4.1 (Pin_1), R1.1, R2.2, SW1.2 (B), U4.2 (GND)
- net at C.1: now also J2.1 (Pin_1), U1.28 (VDD), U1.30 (VDDH), U2.4 (VIN), U2.5 (VBIAS), U3.5 (OUT), J4.2 (Pin_2)
- net at U1.21 (P0.05): now also J1.6 (UART_RX)
- net at U1.22 (P0.06): now also J1.5 (UART_TX)
- net at U1.38 (P0.16): now also U2.6 (ON), R1.2
- net at U1.40 ((reset_configurable)P0.18): now also J4.5 (Pin_5), SW1.1 (A)
- net at U1.41 (P0.17): now also J2.2 (Pin_2), R2.1
- net at U1.51 (SWDIO): now also J4.3 (Pin_3)
- net at U1.53 (SWDCLK): now also J4.4 (Pin_4)
- net at BT.1 (+): now also U3.1 (IN), U3.3 (EN)
- net at U2.1 (VOUT): now also J1.1 (VIN), J3.3 (Pin_3), U4.1 (IN), U4.3 (EN)
- net at J1.3 (1.8V): now also J3.2 (Pin_2), U4.5 (OUT)
- new net: J1.11 (SWD_IO), J3.4 (Pin_4)
- new net: J1.12 (SWD_CLK), J3.5 (Pin_5)
- new net: J1.14 (NRESET), J3.6 (Pin_6)
- new net: J1.23 (DEBUG_UART_TX), J3.7 (Pin_7)
- new net: J1.21 (DEBUG_UART_RX), J3.8 (Pin_8)
- new net: J1.26 (MISC_GPIO2_BOOT0), J3.9 (Pin_9)
Other:
- moved on the sheet: C, J2, U2, U3
