File: hardware/Peripheral_Unit/peripheral-unit.kicad_sch (KiCad schematic)
At the start: 13 parts, among them J1 XM125, J2 EKMB1101111, J3 Conn_01x09, J4 Conn_01x06, SW1 SW_SPST, U1 MDBT50Q-P1M, U2 TPS22860DBVR, U3 TPS7A0233PDBVR, U4 TPS7A0218PDBVR

Commit message: v1.8: Major Fixes
Parts:
- C1: footprint (none) -> Capacitor_Tantalum_SMD:CP_EIA-7343-31_Kemet-D
- J1: footprint (none) -> FDS_library:XM125
- J2: footprint (none) -> FDS_library:EKMB 111001111
- J3: footprint (none) -> Connector_JST:JST_XA_B09B-XASK-1_1x09_P2.50mm_Vertical
- J4: footprint Connector_JST:JST_PH_B6B-PH-K_1x06_P2.00mm_Vertical -> Connector_JST:JST_XA_B08B-XASK-1_1x08_P2.50mm_Vertical
- U2: footprint TPS22860DBVR:SOT95P280X145-6N -> FDS_library:DBV0006A_L
- U3, U4: footprint SOT23_DBV_TEX -> FDS_library:SOT23_DBV_TEX
Changed lines of the file:
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@@
 			)
 		)
-		(property "Footprint" ""
+		(property "Footprint" "Capacitor_Tantalum_SMD:CP_EIA-7343-31_Kemet-D"
 			(at 114.3 65.0748 0)
+			(hide yes)
 			(show_name no)
 			(do_not_autoplace no)
@@
 			)
 		)
-		(property "Footprint" ""
+		(property "Footprint" "Connector_JST:JST_XA_B09B-XASK-1_1x09_P2.50mm_Vertical"
 			(at 246.38 96.52 0)
 			(hide yes)
@@
 			)
 		)
-		(property "Footprint" "Connector_JST:JST_PH_B6B-PH-K_1x06_P2.00mm_Vertical"
+		(property "Footprint" "Connector_JST:JST_XA_B08B-XASK-1_1x08_P2.50mm_Vertical"
 			(at 176.53 22.86 0)
 			(hide yes)
@@
 			)
 		)
-		(property "Description" "Single-cell battery"
+		(property "Description" "ER34615"
 			(at 43.18 42.4814 0)
 			(show_name no)
@@
 				)
 				(justify right)
-			)
-		)
-		(property "Sim.Device" "V"
-			(at 39.37 38.1 0)
-			(hide yes)
-			(show_name no)
-			(do_not_autoplace no)
-			(effects
-				(font
-					(size 1.27 1.27)
-				)
-			)
-		)
-		(property "Sim.Type" "DC"
-			(at 39.37 38.1 0)
-			(hide yes)
-			(show_name no)
-			(do_not_autoplace no)
-			(effects
-				(font
-					(size 1.27 1.27)
-				)
-			)
-		)
-		(property "Sim.Pins" "1=+ 2=-"
-			(at 39.37 38.1 0)
-			(hide yes)
-			(show_name no)
-			(do_not_autoplace no)
-			(effects
-				(font
-					(size 1.27 1.27)
-				)
 			)
 		)
@@
 			)
 		)
-		(property "Footprint" "SOT23_DBV_TEX"
+		(property "Footprint" "FDS_library:SOT23_DBV_TEX"
 			(at 59.182 166.878 0)
 			(hide yes)
@@
 			)
 		)
-		(property "Footprint" "TPS22860DBVR:SOT95P280X145-6N"
+		(property "Footprint" "FDS_library:DBV0006A_L"
 			(at 80.01 143.51 0)
 			(hide yes)
@@
 			)
 		)
-		(property "Footprint" "SOT23_DBV_TEX"
+		(property "Footprint" "FDS_library:SOT23_DBV_TEX"
 			(at 59.69 72.39 0)
 			(hide yes)
@@
 			)
 		)
-		(property "Footprint" ""
+		(property "Footprint" "FDS_library:EKMB 111001111"
 			(at 247.65 124.46 0)
 			(hide yes)
@@
 			)
 		)
-		(property "Footprint" ""
+		(property "Footprint" "FDS_library:XM125"
 			(at 231.14 50.8 0)
-			(show_name no)
-			(do_not_autoplace no)
+			(hide yes)
+			(show_name no)
+			(do_not_autoplace no)

Commit message: Major fixes
Parts:
- BT1: footprint (none) -> Connector_JST:JST_XA_B02B-XASK-1_1x02_P2.50mm_Vertical
- J4: footprint Connector_JST:JST_XA_B08B-XASK-1_1x08_P2.50mm_Vertical -> Connector_JST:JST_XA_B06B-XASK-1_1x06_P2.50mm_Vertical
- R1, R2: footprint (none) -> Resistor_SMD:R_0805_2012Metric
- SW1: footprint (none) -> Button_Switch_SMD:SW_SPST_PTS810
Changed lines of the file:
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@@
 			)
 		)
-		(property "Footprint" ""
+		(property "Footprint" "Resistor_SMD:R_0805_2012Metric"
 			(at 62.23 126.492 90)
 			(hide yes)
@@
 			)
 		)
-		(property "Footprint" "Connector_JST:JST_XA_B08B-XASK-1_1x08_P2.50mm_Vertical"
+		(property "Footprint" "Connector_JST:JST_XA_B06B-XASK-1_1x06_P2.50mm_Vertical"
 			(at 176.53 22.86 0)
 			(hide yes)
@@
 			)
 		)
-		(property "Footprint" ""
+		(property "Footprint" "Connector_JST:JST_XA_B02B-XASK-1_1x02_P2.50mm_Vertical"
 			(at 39.37 39.624 90)
 			(hide yes)
@@
 			)
 		)
-		(property "Footprint" ""
-			(at 195.58 29.21 0)
-			(hide yes)
-			(show_name no)
-			(do_not_autoplace no)
-			(effects
-				(font
-					(size 1.27 1.27)
+		(property "Footprint" "Button_Switch_SMD:SW_SPST_PTS810"
+			(at 194.056 16.002 0)
+			(hide yes)
+			(show_name no)
+			(do_not_autoplace yes)
+			(effects
+				(font
+					(size 1.27 1.27)
+					(thickness 0.1588)
 				)
 			)
@@
 			)
 		)
-		(property "Footprint" ""
+		(property "Footprint" "Resistor_SMD:R_0805_2012Metric"
 			(at 233.172 128.27 90)
 			(hide yes)
