File: hardware/Peripheral_Unit/peripheral-unit.kicad_pcb (KiCad board)
At the start: 2 copper layers, 77 x 37 mm, 13 parts, among them J1 XM125, J2 EKMB1101111, J3 Conn_01x09, J4 Conn_01x06, SW1 SW_SPST, U1 MDBT50Q-P1M, U2 TPS22860DBVR, U3 TPS7A0233PDBVR, U4 TPS7A0218PDBVR

Commit message: Major fixes
Routing:
- net Net-(J2-Pin_2): track 38.2 -> 36.9 mm
- net (no net): vias 0 -> 4
Other:
- board text added: "RESET"
